File: ports_pcb/ports_pcb.kicad_pcb (KiCad board)
At the start: 2 copper layers, 308 x 53.1 mm, 69 parts, among them J1 Conn_01x01_Socket, J10 Conn_01x01_Socket, J100 Joystick, J101 RGB, J102 Printer, J103 Video, J104 Junet, J105 Junet, J106 Tape, J107 5V/2A, J11 Conn_01x01_Socket, J12 Conn_01x01_Socket, J13 Conn_01x01_Socket, J14 Conn_01x01_Socket, J15 Conn_01x01_Socket, J16 Conn_01x01_Socket, J17 Conn_01x01_Socket, J18 Conn_01x01_Socket, J19 Conn_01x01_Socket, J2 Conn_01x01_Socket, J20 Conn_01x01_Socket, J21 Conn_01x01_Socket, J22 Conn_01x01_Socket, J23 Conn_01x01_Socket, J24 Conn_01x01_Socket, J3 Conn_01x01_Socket, J30 Conn_01x01_Socket, J31 Conn_01x01_Socket, J32 Conn_01x01_Socket, J33 Conn_01x01_Socket, J34 Conn_01x01_Socket, J35 Conn_01x01_Socket, J36 Conn_01x01_Socket, J4 Conn_01x01_Socket, J41 RESET1, J42 RESET2, J43 Conn_01x01_Socket, J44 Conn_01x01_Socket, J45 Conn_01x01_Socket, J46 Conn_01x01_Socket, J47 Conn_01x01_Socket, J48 Conn_01x01_Socket, J49 Conn_01x01_Socket, J5 Conn_01x01_Socket, J50 Conn_01x01_Socket, J51 Conn_01x01_Socket, J52 Conn_01x01_Socket, J53 Conn_01x01_Socket, J6 Conn_01x01_Socket, J7 Conn_01x01_Socket, J8 Conn_01x01_Socket, J9 Conn_01x01_Socket, SW1 Reset, SW2 Power

Commit message: Ports PCB: reworked joy (#8) and video (#10)
Parts:
- added JP1: Joy_P8, Connector_PinHeader_2.54mm:PinHeader_1x03_P2.54mm_Vertical, F.Cu at (120.0, 51.0)
- added JP2: SynH, Connector_PinHeader_2.54mm:PinHeader_1x03_P2.54mm_Vertical, F.Cu at (321.9, 52.1)
- added JP3: SynV, Connector_PinHeader_2.54mm:PinHeader_1x02_P2.54mm_Vertical, F.Cu at (348.6, 50.8)
- added R1: 4k7, Resistor_THT:R_Axial_DIN0207_L6.3mm_D2.5mm_P10.16mm_Horizontal, F.Cu at (151.5, 49.9)
- added R2: 4k7, Resistor_THT:R_Axial_DIN0207_L6.3mm_D2.5mm_P10.16mm_Horizontal, F.Cu at (145.5, 49.9)
- added R3: 4k7, Resistor_THT:R_Axial_DIN0207_L6.3mm_D2.5mm_P10.16mm_Horizontal, F.Cu at (139.5, 49.9)
- added R4: 4k7, Resistor_THT:R_Axial_DIN0207_L6.3mm_D2.5mm_P10.16mm_Horizontal, F.Cu at (133.5, 49.9)
- added R5: 4k7, Resistor_THT:R_Axial_DIN0207_L6.3mm_D2.5mm_P10.16mm_Horizontal, F.Cu at (123.5, 45.9)
- added R6: 100, Resistor_THT:R_Axial_DIN0207_L6.3mm_D2.5mm_P10.16mm_Horizontal, F.Cu at (321.9, 48.3)
- added T1: BC557, Package_TO_SOT_THT:TO-92_Inline, F.Cu at (154.4, 54.8)
- added T2: BC557, Package_TO_SOT_THT:TO-92_Inline, F.Cu at (148.4, 54.8)
- added T3: BC557, Package_TO_SOT_THT:TO-92_Inline, F.Cu at (142.5, 54.8)
- added T4: BC557, Package_TO_SOT_THT:TO-92_Inline, F.Cu at (136.4, 54.8)
- added T5: BC557, Package_TO_SOT_THT:TO-92_Inline, F.Cu at (130.4, 54.8)
- J100: footprint Connector_Dsub:DSUB-9_Male_Horizontal_P2.77x2.84mm_EdgePinOffset7.70mm_Housed_MountingHolesOffset9.12mm -> Connector_Dsub:DSUB-9_Pins_Horizontal_P2.77x2.84mm_EdgePinOffset7.70mm_Housed_MountingHolesOffset9.12mm
Connections:
- net Net-(J11-Pin_1) renamed +5V
- net Net-(J9-Pin_1) renamed /j_pwr
- J100 pad 1: /PA3 -> /j_up
- J100 pad 2: /PA2 -> /j_down
- J100 pad 3: /PA1 -> /j_left
- J100 pad 4: /PA0 -> /j_right
- J100 pad 6: /PA4 -> /j_fire
- J100 pad 8: /PA7 -> Net-(JP1-C)
- J101 pad 8: /SYN H -> Net-(JP2-C)
- J101 pad 9: /SYN V -> Net-(JP3-A)
Routing:
- net +5V: track 54.6 -> 131.7 mm
- net /PA6: track 0.00 -> 43.9 mm
- net /PA7: track 42.4 -> 0.00 mm, vias 1 -> 0
- net Net-(JP1-C): track 0.00 -> 28.6 mm
- net /j_fire: track 0.00 -> 27.8 mm
- net Net-(JP2-C): track 0.00 -> 26.5 mm
- net /PA4: track 58.7 -> 33.7 mm
- net /PA3: track 74.6 -> 53.5 mm, vias 0 -> 2
- net /j_pwr: track 39.7 -> 55.8 mm
- net /SYN V: track 61.2 -> 48.1 mm
- net Net-(JP3-A): track 0.00 -> 10.5 mm
- net Net-(T3-B): track 0.00 -> 8.62 mm
- net Net-(T4-B): track 0.00 -> 8.56 mm
- net Net-(T1-B): track 0.00 -> 8.56 mm
- net Net-(T2-B): track 0.00 -> 8.36 mm
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
Commit message: ports_pcb: added fuse, aux power connector, changed DIN 3d model
Parts:
- added C1: 100nF, Capacitor_THT:C_Disc_D5.0mm_W2.5mm_P2.50mm, F.Cu at (318.8, 48.2)
- added F1: 2A, Fuse:Fuseholder_Clip-5x20mm_Littelfuse_445-030_Inline_P20.50x5.20mm_D1.30mm_Horizontal, F.Cu at (399.7, 54.4)
- added J108: Conn_01x02, Connector_Molex:Molex_KK-254_AE-6410-02A_1x02_P2.54mm_Vertical, F.Cu at (383.5, 48.9)
- added kibuzzard-67F7609F: G***, kibuzzard-67F7609F, F.Cu at (339.6, 50.5)
- added kibuzzard-67F760B8: G***, kibuzzard-67F760B8, F.Cu at (367.3, 54.5)
- added kibuzzard-67F76112: G***, kibuzzard-67F76112, F.Cu at (305.8, 54.5)
- added kibuzzard-67F762C8: G***, kibuzzard-67F762C8, F.Cu at (253.9, 54.5)
- added kibuzzard-67F762C8: G***, kibuzzard-67F762C8, F.Cu at (233.7, 54.5)
- added kibuzzard-67F763AC: G***, kibuzzard-67F763AC, F.Cu at (203.8, 50.5)
- added kibuzzard-67F76475: G***, kibuzzard-67F76475, F.Cu at (158.8, 43.2)
- added kibuzzard-67F78920: G***, kibuzzard-67F78920, F.Cu at (418.1, 45.8)
- J101: footprint Connector_Dsub:DSUB-9_Female_Horizontal_P2.77x2.84mm_EdgePinOffset7.70mm_Housed_MountingHolesOffset9.12mm -> Connector_Dsub:DSUB-9_Socket_Horizontal_P2.77x2.84mm_EdgePinOffset7.70mm_Housed_MountingHolesOffset9.12mm
- J102: footprint Connector_Dsub:DSUB-25_Female_Horizontal_P2.77x2.84mm_EdgePinOffset7.70mm_Housed_MountingHolesOffset9.12mm -> Connector_Dsub:DSUB-25_Socket_Horizontal_P2.77x2.84mm_EdgePinOffset7.70mm_Housed_MountingHolesOffset9.12mm
- moved T3 0.14 mm to (142.4, 54.7)
Connections:
- J107 pad 1: Net-(J107-Pad1) -> Net-(F1-Pad2)
- SW2 pad 2: Net-(J107-Pad1) -> Net-(F1-Pad1)
- SW2 pad 5: Net-(J107-Pad1) -> Net-(F1-Pad1)
Routing:
- net Net-(J107-Pad1): track 22.8 -> 0.00 mm
- net Net-(F1-Pad1): track 0.00 -> 19.2 mm
- net Net-(F1-Pad2): track 0.00 -> 14.5 mm
- net /j_pwr: track 55.8 -> 64.7 mm
- net Net-(JP2-A): track 3.81 -> 6.99 mm
- net /SYN H: track 74.7 -> 77.3 mm
- net GND: vias 55 -> 54
Other:
- board text added: "+5V"
- board text added: "Elwro 800 Junior replica port breakout PCB v1.1 https://e800j.codepainters.com/ pwegrzyn@codepainters.com"
- board text added: "GND"
- board text added: "P8"
- board text added: "P9"
- board text added: "SYN H"
- board text added: "SYN V"
- board text removed: "Elwro 800 Junior replica port breakout PCB v1.0 https://e800j.codepainters.com/ pwegrzyn@codepainters.com"

Commit message: ports_pcb: labels replaced with thicker font (#11)
Parts:
- removed kibuzzard-67F7609F: G***, kibuzzard-67F7609F
- removed kibuzzard-67F760B8: G***, kibuzzard-67F760B8
- removed kibuzzard-67F76112: G***, kibuzzard-67F76112
- removed kibuzzard-67F762C8 (x2): G***, kibuzzard-67F762C8
- removed kibuzzard-67F763AC: G***, kibuzzard-67F763AC
- removed kibuzzard-67F76475: G***, kibuzzard-67F76475
- removed kibuzzard-67F78920: G***, kibuzzard-67F78920
- added kibuzzard-67F8F98E: G***, kibuzzard-67F8F98E, F.Cu at (339.6, 50.5)
- added kibuzzard-67F9119B: G***, kibuzzard-67F9119B, F.Cu at (158.8, 43.9)
- added kibuzzard-67F911BA: G***, kibuzzard-67F911BA, F.Cu at (206.0, 50.5)
- added kibuzzard-67F911F0: G***, kibuzzard-67F911F0, F.Cu at (254.0, 54.6)
- added kibuzzard-67F911F0: G***, kibuzzard-67F911F0, F.Cu at (233.7, 54.6)
- added kibuzzard-67F91269: G***, kibuzzard-67F91269, F.Cu at (305.8, 54.6)
- added kibuzzard-67F91296: G***, kibuzzard-67F91296, F.Cu at (367.3, 54.6)
- added kibuzzard-67F91771: G***, kibuzzard-67F91771, F.Cu at (418.0, 45.5)
