File: ports_pcb/ports_pcb.kicad_pcb (KiCad board)
At the start: 2 copper layers, 308 x 53.1 mm, 94 parts, among them J1 Conn_01x01_Socket, J10 Conn_01x01_Socket, J100 Joystick, J101 RGB, J102 Printer, J103 Video, J104 Junet, J105 Junet, J106 Tape, J107 5V/2A, J108 Conn_01x02, J11 Conn_01x01_Socket, J12 Conn_01x01_Socket, J13 Conn_01x01_Socket, J14 Conn_01x01_Socket, J15 Conn_01x01_Socket, J16 Conn_01x01_Socket, J17 Conn_01x01_Socket, J18 Conn_01x01_Socket, J19 Conn_01x01_Socket, J2 Conn_01x01_Socket, J20 Conn_01x01_Socket, J21 Conn_01x01_Socket, J22 Conn_01x01_Socket, J23 Conn_01x01_Socket, J24 Conn_01x01_Socket, J3 Conn_01x01_Socket, J30 Conn_01x01_Socket, J31 Conn_01x01_Socket, J32 Conn_01x01_Socket, J33 Conn_01x01_Socket, J34 Conn_01x01_Socket, J35 Conn_01x01_Socket, J36 Conn_01x01_Socket, J4 Conn_01x01_Socket, J41 RESET1, J42 RESET2, J43 Conn_01x01_Socket, J44 Conn_01x01_Socket, J45 Conn_01x01_Socket, J46 Conn_01x01_Socket, J47 Conn_01x01_Socket, J48 Conn_01x01_Socket, J49 Conn_01x01_Socket, J5 Conn_01x01_Socket, J50 Conn_01x01_Socket, J51 Conn_01x01_Socket, J52 Conn_01x01_Socket, J53 Conn_01x01_Socket, J6 Conn_01x01_Socket, J7 Conn_01x01_Socket, J8 Conn_01x01_Socket, J9 Conn_01x01_Socket, SW1 Reset, SW2 Power, T1 BC557, T2 BC557, T3 BC557, T4 BC557, T5 BC557

Commit message: ports_pcb: excluded Jx headers from BOM
Parts:
- renumbered REF** to IMG1
Changed lines of the file:
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@@
 		(sheetname "/")
 		(sheetfile "ports_pcb.kicad_sch")
-		(attr through_hole)
+		(attr through_hole exclude_from_bom)
 		(fp_line
 			(start -1.38 -1.38)
@@
 		(sheetname "/")
 		(sheetfile "ports_pcb.kicad_sch")
-		(attr through_hole)
+		(attr through_hole exclude_from_bom)
 		(fp_line
 			(start -1.38 -1.38)
@@
 		(sheetname "/")
 		(sheetfile "ports_pcb.kicad_sch")
-		(attr through_hole)
+		(attr through_hole exclude_from_bom)
 		(fp_line
 			(start -1.38 -1.38)
@@
 		(sheetname "/")
 		(sheetfile "ports_pcb.kicad_sch")
-		(attr through_hole)
+		(attr through_hole exclude_from_bom)
 		(fp_circle
 			(center 0 0)
@@
 		(sheetname "/")
 		(sheetfile "ports_pcb.kicad_sch")
-		(attr through_hole)
+		(attr through_hole exclude_from_bom)
 		(fp_circle
 			(center 0 0)
@@
 		(sheetname "/")
 		(sheetfile "ports_pcb.kicad_sch")
-		(attr through_hole)
+		(attr through_hole exclude_from_bom)
 		(fp_line
 			(start -1.38 -1.38)
@@
 		(sheetname "/")
 		(sheetfile "ports_pcb.kicad_sch")
-		(attr through_hole)
+		(attr through_hole exclude_from_bom)
 		(fp_line
 			(start -1.38 -1.38)
@@
 		(sheetname "/")
 		(sheetfile "ports_pcb.kicad_sch")
-		(attr through_hole)
+		(attr through_hole exclude_from_bom)
 		(fp_line
 			(start -1.38 -1.38)
@@
 		(sheetname "/")
 		(sheetfile "ports_pcb.kicad_sch")
-		(attr through_hole)
+		(attr through_hole exclude_from_bom)
 		(fp_line
 			(start -1.38 -1.38)
@@
 		(sheetname "/")
 		(sheetfile "ports_pcb.kicad_sch")
-		(attr through_hole)
+		(attr through_hole exclude_from_bom)
 		(fp_line
 			(start -1.38 -1.38)
@@
 		(sheetname "/")
 		(sheetfile "ports_pcb.kicad_sch")
-		(attr through_hole)
+		(attr through_hole exclude_from_bom)
 		(fp_line
 			(start -1.38 -1.38)
@@
 		(sheetname "/")
 		(sheetfile "ports_pcb.kicad_sch")
-		(attr through_hole)
+		(attr through_hole exclude_from_bom)
 		(fp_line
 			(start -1.38 -1.38)
@@
 		(sheetname "/")
 		(sheetfile "ports_pcb.kicad_sch")
-		(attr through_hole)
+		(attr through_hole exclude_from_bom)
 		(fp_line
 			(start -1.38 -1.38)
@@
 		(layer "F.Cu")
 		(at 266.065 73.66)
-		(property "Reference" "REF**"
+		(property "Reference" "IMG1"
 			(at 1.508317 0.53122 0)
 			(unlocked yes)
@@
 			)
 		)
-		(attr smd board_only)
+		(attr smd board_only exclude_from_bom)
 		(fp_poly
 			(pts
@@
 		(sheetname "/")
 		(sheetfile "ports_pcb.kicad_sch")
-		(attr through_hole)
+		(attr through_hole exclude_from_bom)
 		(fp_line
 			(start -1.38 -1.38)
@@
 		(sheetname "/")
 		(sheetfile "ports_pcb.kicad_sch")
-		(attr through_hole)
+		(attr through_hole exclude_from_bom)
 		(fp_line
 			(start -1.38 -1.38)
@@
 		(sheetname "/")
 		(sheetfile "ports_pcb.kicad_sch")
-		(attr through_hole)
+		(attr through_hole exclude_from_bom)
 		(fp_circle
 			(center 0 0)
@@
 		(sheetname "/")
 		(sheetfile "ports_pcb.kicad_sch")
-		(attr through_hole)
+		(attr through_hole exclude_from_bom)
 		(fp_line
 			(start -1.38 -1.38)
@@
 		(sheetname "/")
 		(sheetfile "ports_pcb.kicad_sch")
-		(attr through_hole)
+		(attr through_hole exclude_from_bom)
 		(fp_circle
 			(center 0 0)
@@
 		(sheetname "/")
 		(sheetfile "ports_pcb.kicad_sch")
-		(attr through_hole)
+		(attr through_hole exclude_from_bom)
 		(fp_line
 			(start -1.38 -1.38)
@@
 		(sheetname "/")
 		(sheetfile "ports_pcb.kicad_sch")
-		(attr through_hole)
+		(attr through_hole exclude_from_bom)
 		(fp_line
 			(start -1.38 -1.38)
@@
 		(sheetname "/")
 		(sheetfile "ports_pcb.kicad_sch")
-		(attr through_hole)
+		(attr through_hole exclude_from_bom)
 		(fp_line
 			(start -1.38 -1.38)
@@
 		(sheetname "/")
 		(sheetfile "ports_pcb.kicad_sch")
-		(attr through_hole)
+		(attr through_hole exclude_from_bom)
 		(fp_line
 			(start -1.38 -1.38)
@@
 		(sheetname "/")
 		(sheetfile "ports_pcb.kicad_sch")
-		(attr through_hole)
+		(attr through_hole exclude_from_bom)
 		(fp_line
 			(start -1.38 -1.38)
@@
 		(sheetname "/")
 		(sheetfile "ports_pcb.kicad_sch")
-		(attr through_hole)
+		(attr through_hole exclude_from_bom)
 		(fp_line
 			(start -1.38 -1.38)
@@
 		(sheetname "/")
 		(sheetfile "ports_pcb.kicad_sch")
-		(attr through_hole)
+		(attr through_hole exclude_from_bom)
 		(fp_line
 			(start -1.38 -1.38)
@@
 		(sheetname "/")
 		(sheetfile "ports_pcb.kicad_sch")
-		(attr through_hole)
+		(attr through_hole exclude_from_bom)
 		(fp_line
 			(start -1.38 -1.38)
@@
 		(sheetname "/")
 		(sheetfile "ports_pcb.kicad_sch")
-		(attr through_hole)
+		(attr through_hole exclude_from_bom)
 		(fp_line
 			(start -1.38 -1.38)
@@
 		(sheetname "/")
 		(sheetfile "ports_pcb.kicad_sch")
-		(attr through_hole)
+		(attr through_hole exclude_from_bom)
 		(fp_line
 			(start -1.38 -1.38)
@@
 		(sheetname "/")
 		(sheetfile "ports_pcb.kicad_sch")
-		(attr through_hole)
+		(attr through_hole exclude_from_bom)
 		(fp_line
 			(start -1.38 -1.38)
@@
 		(sheetname "/")
 		(sheetfile "ports_pcb.kicad_sch")
-		(attr through_hole)
+		(attr through_hole exclude_from_bom)
 		(fp_line
 			(start -1.38 -1.38)
@@
 		(sheetname "/")
 		(sheetfile "ports_pcb.kicad_sch")
-		(attr through_hole)
+		(attr through_hole exclude_from_bom)
 		(fp_line
 			(start -1.38 -1.38)
@@
 		(sheetname "/")
 		(sheetfile "ports_pcb.kicad_sch")
-		(attr through_hole)
+		(attr through_hole exclude_from_bom)
 		(fp_line
 			(start -1.38 -1.38)
@@
 		(sheetname "/")
 		(sheetfile "ports_pcb.kicad_sch")
-		(attr through_hole)
+		(attr through_hole exclude_from_bom)
 		(fp_line
 			(start -1.38 -1.38)
@@
 		(sheetname "/")
 		(sheetfile "ports_pcb.kicad_sch")
-		(attr through_hole)
+		(attr through_hole exclude_from_bom)
 		(fp_line
 			(start -1.38 -1.38)
@@
 		(sheetname "/")
 		(sheetfile "ports_pcb.kicad_sch")
-		(attr through_hole)
+		(attr through_hole exclude_from_bom)
 		(fp_line
 			(start -1.38 -1.38)
@@
 		(sheetname "/")
 		(sheetfile "ports_pcb.kicad_sch")
-		(attr through_hole)
+		(attr through_hole exclude_from_bom)
 		(fp_line
 			(start -1.38 -1.38)
@@
 		(sheetname "/")
 		(sheetfile "ports_pcb.kicad_sch")
-		(attr through_hole)
+		(attr through_hole exclude_from_bom)
 		(fp_line
 			(start -1.38 -1.38)
@@
 		(sheetname "/")
 		(sheetfile "ports_pcb.kicad_sch")
-		(attr through_hole)
+		(attr through_hole exclude_from_bom)
 		(fp_line
 			(start -1.38 -1.38)
@@
 		(sheetname "/")
 		(sheetfile "ports_pcb.kicad_sch")
-		(attr through_hole)
+		(attr through_hole exclude_from_bom)
 		(fp_line
 			(start -1.38 -1.38)
@@
 		(sheetname "/")
 		(sheetfile "ports_pcb.kicad_sch")
-		(attr through_hole)
+		(attr through_hole exclude_from_bom)
 		(fp_line
 			(start -1.38 -1.38)
@@
 		(sheetname "/")
 		(sheetfile "ports_pcb.kicad_sch")
-		(attr through_hole)
+		(attr through_hole exclude_from_bom)
 		(fp_line
 			(start -1.38 -1.38)
@@
 		(sheetname "/")
 		(sheetfile "ports_pcb.kicad_sch")
-		(attr through_hole)
+		(attr through_hole exclude_from_bom)
 		(fp_line
 			(start -1.38 -1.38)
@@
 		(sheetname "/")
 		(sheetfile "ports_pcb.kicad_sch")
-		(attr through_hole)
+		(attr through_hole exclude_from_bom)
 		(fp_line
 			(start -1.38 -1.38)
@@
 		(sheetname "/")
 		(sheetfile "ports_pcb.kicad_sch")
-		(attr through_hole)
+		(attr through_hole exclude_from_bom)
 		(fp_line
 			(start -1.38 -1.38)
@@
 		(sheetname "/")
 		(sheetfile "ports_pcb.kicad_sch")
-		(attr through_hole)
+		(attr through_hole exclude_from_bom)
 		(fp_line
 			(start -1.38 -1.38)
@@
 		(sheetname "/")
 		(sheetfile "ports_pcb.kicad_sch")
-		(attr through_hole)
+		(attr through_hole exclude_from_bom)
 		(fp_circle
 			(center 0 0)
@@
 		(sheetname "/")
 		(sheetfile "ports_pcb.kicad_sch")
-		(attr through_hole)
+		(attr through_hole exclude_from_bom)
 		(fp_line
 			(start -1.38 -1.38)
@@
 		(sheetname "/")
 		(sheetfile "ports_pcb.kicad_sch")
-		(attr through_hole)
+		(attr through_hole exclude_from_bom)
 		(fp_line
 			(start -1.38 -1.38)

Commit message: ports_pcb: added jP4 jumper to allow disconnecting FON (#13)
Parts:
- added JP4: FON, Connector_PinHeader_2.54mm:PinHeader_1x02_P2.54mm_Vertical, F.Cu at (318.1, 41.7)
- R6: value 100 -> 0R*
- moved C1 1.44 mm to (318.1, 49.5), turned to -90 degrees
Connections:
- J101 pad 7: /FON -> Net-(JP4-B)
Routing:
- net Net-(JP4-B): track 0.00 -> 23.1 mm
- net /FON: track 266.9 -> 263.3 mm
- net Net-(JP2-A): track 6.99 -> 8.16 mm
Other:
- board text added: "P7"

Commit message: prots_pcb: minor tweaks, v1.2
Other:
- board text added: "Elwro 800 Junior replica port breakout PCB v1.2 https://e800j.codepainters.com/ pwegrzyn@codepainters.com"
- board text removed: "Elwro 800 Junior replica port breakout PCB v1.1 https://e800j.codepainters.com/ pwegrzyn@codepainters.com"
Changed lines of the file:
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@@
 		(layer "Edge.Cuts")
 	)
-	(gr_text "Elwro 800 Junior replica \nport breakout PCB v1.1\n\nhttps://e800j.codepainters.com/\npwegrzyn@codepainters.com"
+	(gr_text "Elwro 800 Junior replica \nport breakout PCB v1.2\n\nhttps://e800j.codepainters.com/\npwegrzyn@codepainters.com"
 		(at 342.9 82.55 0)
 		(layer "F.SilkS")
@@
 	)
 	(segment
-		(start 146.05 71.501)
-		(end 149.301 68.25)
-		(width 0.6096)
-		(layer "B.Cu")
-		(net 38)
-	)
-	(segment
-		(start 299.085 40.64)
-		(end 314.325 40.64)
-		(width 0.6096)
-		(layer "B.Cu")
-		(net 38)
-	)
-	(segment
-		(start 276.86 38.735)
-		(end 297.18 38.735)
+		(start 372.919 48.434)
+		(end 374.738 48.434)
 		(width 0.6096)
 		(layer "B.Cu")
@@
 	)
 	(segment
-		(start 151.25 68.25)
-		(end 159.385 60.115)
+		(start 325.12 40.005)
+		(end 353.06 40.005)
 		(width 0.6096)
 		(layer "B.Cu")
@@
 	)
 	(segment
-		(start 267.335 43.815)
-		(end 271.78 43.815)
+		(start 146.05 71.501)
+		(end 149.301 68.25)
 		(width 0.6096)
 		(layer "B.Cu")
@@
 	)
 	(segment
-		(start 271.78 43.815)
-		(end 276.86 38.735)
+		(start 299.085 40.64)
+		(end 314.6425 40.64)
 		(width 0.6096)
 		(layer "B.Cu")
@@
 	)
 	(segment
-		(start 325.12 40.005)
-		(end 340.743 40.005)
+		(start 223.52 40.64)
+		(end 264.16 40.64)
 		(width 0.6096)
 		(layer "B.Cu")
@@
 	)
 	(segment
-		(start 159.385 60.115)
-		(end 159.385 41.275)
+		(start 146.05 72.39)
+		(end 146.05 71.501)
 		(width 0.6096)
 		(layer "B.Cu")
@@
 	)
 	(segment
-		(start 323.469 41.656)
-		(end 325.12 40.005)
+		(start 276.86 38.735)
+		(end 297.18 38.735)
 		(width 0.6096)
 		(layer "B.Cu")
@@
 	)
 	(segment
-		(start 264.16 40.64)
-		(end 267.335 43.815)
+		(start 370.205 45.72)
+		(end 372.919 48.434)
 		(width 0.6096)
 		(layer "B.Cu")
@@
 	)
 	(segment
-		(start 315.341 41.656)
+		(start 315.6585 41.656)
 		(end 323.469 41.656)
 		(width 0.6096)
@@
 	)
 	(segment
-		(start 146.05 72.39)
-		(end 146.05 71.501)
+		(start 149.301 68.25)
+		(end 151.25 68.25)
 		(width 0.6096)
 		(layer "B.Cu")
@@
 	)
 	(segment
-		(start 297.18 38.735)
-		(end 299.085 40.64)
+		(start 358.775 45.72)
+		(end 370.205 45.72)
 		(width 0.6096)
 		(layer "B.Cu")
@@
 	)
 	(segment
-		(start 149.301 68.25)
-		(end 151.25 68.25)
+		(start 264.16 40.64)
+		(end 267.335 43.815)
 		(width 0.6096)
 		(layer "B.Cu")
@@
 	)
 	(segment
-		(start 223.52 40.64)
-		(end 264.16 40.64)
+		(start 151.25 68.25)
+		(end 159.385 60.115)
 		(width 0.6096)
 		(layer "B.Cu")
@@
 	)
 	(segment
-		(start 358.775 45.72)
-		(end 370.205 45.72)
+		(start 159.385 60.115)
+		(end 159.385 41.275)
 		(width 0.6096)
 		(layer "B.Cu")
@@
 	)
 	(segment
-		(start 340.743 40.005)
-		(end 341.378 40.64)
+		(start 159.385 41.275)
+		(end 161.29 39.37)
 		(width 0.6096)
 		(layer "B.Cu")
@@
 	)
 	(segment
-		(start 314.325 40.64)
-		(end 315.341 41.656)
+		(start 222.25 39.37)
+		(end 223.52 40.64)
 		(width 0.6096)
 		(layer "B.Cu")
@@
 	)
 	(segment
-		(start 159.385 41.275)
-		(end 161.29 39.37)
+		(start 297.18 38.735)
+		(end 299.085 40.64)
 		(width 0.6096)
 		(layer "B.Cu")
@@
 	)
 	(segment
-		(start 372.919 48.434)
-		(end 374.738 48.434)
+		(start 353.06 40.005)
+		(end 358.775 45.72)
 		(width 0.6096)
 		(layer "B.Cu")
@@
 	)
 	(segment
-		(start 341.378 40.64)
-		(end 353.695 40.64)
+		(start 323.469 41.656)
+		(end 325.12 40.005)
 		(width 0.6096)
 		(layer "B.Cu")
@@
 	)
 	(segment
-		(start 222.25 39.37)
-		(end 223.52 40.64)
+		(start 267.335 43.815)
+		(end 271.78 43.815)
 		(width 0.6096)
 		(layer "B.Cu")
@@
 	)
 	(segment
-		(start 370.205 45.72)
-		(end 372.919 48.434)
+		(start 314.6425 40.64)
+		(end 315.6585 41.656)
 		(width 0.6096)
 		(layer "B.Cu")
@@
 	)
 	(segment
-		(start 353.695 40.64)
-		(end 358.775 45.72)
+		(start 271.78 43.815)
+		(end 276.86 38.735)
 		(width 0.6096)
 		(layer "B.Cu")
@@
 	)
 	(segment
-		(start 318.384 44.445)
-		(end 318.135 44.196)
-		(width 0.6096)
-		(layer "B.Cu")
-		(net 76)
-	)
-	(segment
-		(start 320.67 44.445)
-		(end 318.384 44.445)
+		(start 337.185 41.275)
+		(end 325.755 41.275)
 		(width 0.6096)
 		(layer "B.Cu")
@@
 	)
 	(segment
-		(start 337.185 41.275)
-		(end 325.755 41.275)
+		(start 324.104 42.926)
+		(end 320.929 42.926)
 		(width 0.6096)
 		(layer "B.Cu")
@@
 	)
 	(segment
-		(start 320.675 44.45)
-		(end 320.67 44.445)
+		(start 319.659 44.196)
+		(end 318.135 44.196)
 		(width 0.6096)
 		(layer "B.Cu")
@@
 	)
 	(segment
-		(start 321.31 43.815)
-		(end 320.675 44.45)
+		(start 338.203 43.434)
+		(end 338.203 42.293)
 		(width 0.6096)
 		(layer "B.Cu")
@@
 	)
 	(segment
-		(start 338.203 43.434)
-		(end 338.203 42.293)
+		(start 320.929 42.926)
+		(end 319.659 44.196)
 		(width 0.6096)
 		(layer "B.Cu")
@@
 	(segment
 		(start 325.755 41.275)
-		(end 323.215 43.815)
-		(width 0.6096)
-		(layer "B.Cu")
-		(net 76)
-	)
-	(segment
-		(start 323.215 43.815)
-		(end 321.31 43.815)
+		(end 324.104 42.926)
 		(width 0.6096)
 		(layer "B.Cu")
