File: kbd_cherry/kbd_cherry.kicad_sch (KiCad schematic)
At the start: 79 parts, among them SW1 ^-, SW10 H, SW11 J, SW12 K, SW13 L, SW14 CR, SW15 BS, SW16 ESC, SW17 Y, SW18 U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

Commit message: kbd_cherry: converted to KiCAD 9, schematic size reduced to A4
Other:
- company: (none) -> Przemysław Węgrzyn <pwegrzyn@codepainters.com>
- title: (none) -> Elwro 800 Junior replica - Cherry MX keyboard
- moved on the sheet: D1, G1, G2, SW1, SW10, SW11, SW12, SW13, SW14, SW15, SW16, SW17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
