File: e800j_rev_c/junet.kicad_sch (KiCad schematic)
At the start: 33 parts, among them T6 BD135, T7 BD135, T8 BD135, U21 74LS00, U60 74LS04, U61 8251, U67 74132, U70 74LS74

Commit message: mianboard: more fixes (#3, #4, #6)
- #3 - fixed GWP10 (keyboard connector) footprint pitch
- #4 - increased Z3 jumper hole diameters
- #6 - increased silkscreen circles diameter and thickness
Parts:
- Z3: footprint e800j_custom:jmp_100 -> e800j_custom:jmp_100_idc
Changed lines of the file:
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@@
 		(mirror x)
 		(unit 1)
-		(exclude_from_sim yes)
+		(exclude_from_sim no)
 		(in_bom yes)
 		(on_board yes)
@@
 			)
 		)
-		(property "Footprint" "e800j_custom:jmp_100"
+		(property "Footprint" "e800j_custom:jmp_100_idc"
 			(at 111.76 160.02 0)
 			(effects
