File: e800j_rev_c/pio.kicad_sch (KiCad schematic)
At the start: 35 parts, among them J1 Conn_01x01_Socket, J10 Conn_01x01_Socket, J14 Conn_01x01_Socket, J15 Conn_01x01_Socket, J16 Conn_01x01_Socket, J17 Conn_01x01_Socket, J18 Conn_01x01_Socket, J19 Conn_01x01_Socket, J2 Conn_01x01_Socket, J20 Conn_01x01_Socket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

Commit message: mainboard: minor fixes
Parts:
- JMP1: now left out of the parts list
Changed lines of the file:
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@@
 		(at 156.21 66.04 0)
 		(unit 1)
-		(exclude_from_sim yes)
-		(in_bom yes)
+		(exclude_from_sim no)
+		(in_bom no)
 		(on_board yes)
 		(dnp no)
