File: e800j_rev_c/video.kicad_sch (KiCad schematic)
At the start: 63 parts, among them J43 Conn_01x01_Socket, J44 Conn_01x01_Socket, J45 Conn_01x01_Socket, J46 Conn_01x01_Socket, J47 Conn_01x01_Socket, J48 Conn_01x01_Socket, J49 Conn_01x01_Socket, J50 Conn_01x01_Socket, J51 Conn_01x01_Socket, J52 Conn_01x01_Socket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

Commit message: mainboard: minor fixes
Parts:
- Z2: now left out of the parts list
Changed lines of the file:
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@@
 		(mirror x)
 		(unit 1)
-		(exclude_from_sim yes)
-		(in_bom yes)
+		(exclude_from_sim no)
+		(in_bom no)
 		(on_board yes)
 		(dnp no)
