File: e800j_rev_c/power.kicad_sch (KiCad schematic)
At the start: 86 parts, among them J11 Conn_01x01_Socket, J12 Conn_01x01_Socket, J13 Conn_01x01_Socket, U1 74LS04, U11 74LS00, U12 7438, U18 74LS02, U21 74LS00, U3 74LS32, U4 74LS04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

Commit message: Marked unpopulated components properly (see #14)
Parts:
- U5: now left out of the parts list
Changed lines of the file:
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@@
 		(unit 2)
 		(exclude_from_sim no)
-		(in_bom yes)
+		(in_bom no)
 		(on_board yes)
 		(dnp no)
@@
 		(unit 6)
 		(exclude_from_sim no)
-		(in_bom yes)
+		(in_bom no)
 		(on_board yes)
 		(dnp no)
@@
 		(unit 1)
 		(exclude_from_sim no)
-		(in_bom yes)
+		(in_bom no)
 		(on_board yes)
 		(dnp no)
@@
 		(unit 7)
 		(exclude_from_sim no)
-		(in_bom yes)
+		(in_bom no)
 		(on_board yes)
 		(dnp no)
